Commit message: Scaling change in mocap system

File: superchick/motionCaptureSystem.xacro (robot description, xacro)
@@ -12,5 +12,5 @@
       <origin xyz="0 0 0" rpy="${PI/2} 0 ${PI/2}" />
       <geometry>
-        <mesh filename="package://superchick/meshes/motionCapture.stl" scale = ".001 .001 .001" />
+        <mesh filename="package://superchick/meshes/motionCapture.stl" scale = ".000001 .000001 .000001" />
       </geometry>
     </visual>
@@ -18,5 +18,5 @@
       <origin xyz="0 0 0" rpy="${PI/2} 0 ${PI/2}" />
       <geometry>
-        <mesh filename="package://superchick/meshes/motionCapture.stl" scale = ".001 .001 .001" />
+        <mesh filename="package://superchick/meshes/motionCapture.stl" scale = ".000001 .000001 .000001" />
       </geometry>
     </collision>

Commit message: Alex--Vicon dependencies changes

File: superchick/motionCaptureSystem.xacro (robot description, xacro)
@@ -12,5 +12,5 @@
       <origin xyz="0 0 0" rpy="${PI/2} 0 ${PI/2}" />
       <geometry>
-        <mesh filename="package://superchick/meshes/motionCapture.stl" scale = ".000001 .000001 .000001" />
+        <mesh filename="package://superchick/meshes/motionCapture.stl" scale = ".001 .001 .001" />
       </geometry>
     </visual>
@@ -18,5 +18,5 @@
       <origin xyz="0 0 0" rpy="${PI/2} 0 ${PI/2}" />
       <geometry>
-        <mesh filename="package://superchick/meshes/motionCapture.stl" scale = ".000001 .000001 .000001" />
+        <mesh filename="package://superchick/meshes/motionCapture.stl" scale = ".001 .001 .001" />
       </geometry>
     </collision>
