Commit message: updates to work

File: superchick/superchick.urdf (robot description, URDF)
Before this commit: robot superchick, 12 links, 12 joints
Links:
- link big_bladder_link: geometry visual box size=0.31496 0.31496 0.0508
- link headnball_link: geometry visual mesh filename=package://superchick/meshes/headnball.stl scale=.001 .001 .001
